File: eagle/Mega Shield/Mega_Shield-v13.brd (EAGLE design)
At the start: 113 x 96.5 mm, 51 parts, among them Q1 2N3904, Q2 2N3904, Q4 2N3904, Q5 2N3906

Commit message: ordered pcbs
Parts:
- removed ABOX_HARN, DSW_LG: (no value), Molex connectors:172064-0012
- added ABOX_HARN_0, ABOX_HARN_1, ABOX_HARN_2, ABOX_HARN_3, DSW_LG_0, DSW_LG_1, DSW_LG_2: 5569, MHR14:5569
- added JP20, JP21, JP22, JP23, JP24, JP25, JP26, JP27: M12PTH, SparkFun-Connectors:1X12
- added U$1: (no value), MHR14:BLOCKM
- ABOX_PWR, DSW_SM, STEER: value (none) -> 5569; device Molex connectors:172064-0004 -> MHR14:5569
- moved STEER 97.7 mm to (0.00, 34.3), turned to 270 degrees
- moved R12 42.0 mm to (31.8, 31.8), turned to 90 degrees
- moved DSW_SM 42.0 mm to (68.6, 88.9)
- moved R14 39.7 mm to (39.4, 31.8), turned to 90 degrees
- moved R13 37.5 mm to (29.2, 31.8), turned to 90 degrees
- moved R15 33.5 mm to (34.3, 31.8), turned to 90 degrees
- moved R16 32.3 mm to (36.8, 31.8), turned to 270 degrees
- moved ABOX_PWR 8.13 mm to (0.00, 24.1)
- moved JP11 6.35 mm to (100.3, 15.2)
- moved JP12 6.35 mm to (100.3, 58.4)
- moved JP16 6.35 mm to (110.5, 17.8)
- moved JP2 6.35 mm to (69.8, 63.5)
- moved JP4 6.35 mm to (69.8, 58.4)
- moved JP9 6.35 mm to (100.3, 55.9)
- moved LCD_0 6.35 mm to (83.8, 28.6)
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Connections:
- removed net N$98: DSW_SM.CKT2
- removed net N$99: DSW_SM.CKT1
- new net E_DSEN_LED: ABOX_HARN_3.CKT2, DSW_SM.CKT2
- new net E_DSEN_SW: ABOX_HARN_3.CKT3, STEER.CKT2
- new net GFD_LED: ABOX_HARN_3.CKT1, DSW_SM.CKT1
- net 5V: now also JP20.12, JP21.12, JP22.12, JP23.12, JP24.12, JP25.12, JP26.12, JP27.12
- net A7: now also ABOX_HARN_3.CKT4
- net D24: now also DSW_LG_1.CKT2; no longer DSW_LG.CKT6
- net GND: now also JP20.1, JP21.1, JP22.1, JP23.1, JP24.1, JP25.1, JP26.1, JP27.1; no longer STEER.CKT2
- net LAUNCHSW_12: now also DSW_LG_0.CKT2; no longer DSW_LG.CKT2
- net LAUNCHSW_LED: now also DSW_LG_0.CKT3; no longer DSW_LG.CKT3
- net LAUNCH_LED: now also ABOX_HARN_2.CKT3; no longer ABOX_HARN.CKT11
- net LAUNCH_SW: now also ABOX_HARN_1.CKT4; no longer ABOX_HARN.CKT8
- net MODE0: now also ABOX_HARN_1.CKT2, DSW_LG_1.CKT4; no longer ABOX_HARN.CKT6, DSW_LG.CKT8
- net MODE1: now also ABOX_HARN_1.CKT3, DSW_LG_2.CKT1; no longer ABOX_HARN.CKT7, DSW_LG.CKT9
- net SERIAL_K: now also ABOX_HARN_0.CKT1; no longer ABOX_HARN.CKT1
- net SERIAL_L: now also ABOX_HARN_0.CKT2; no longer ABOX_HARN.CKT2
- net SW1: now also ABOX_HARN_0.CKT3, DSW_LG_2.CKT2; no longer ABOX_HARN.CKT3, DSW_LG.CKT10
- net SW2: now also ABOX_HARN_0.CKT4, DSW_LG_2.CKT3; no longer ABOX_HARN.CKT4, DSW_LG.CKT11
- net SW3: now also ABOX_HARN_1.CKT1, DSW_LG_2.CKT4; no longer ABOX_HARN.CKT5, DSW_LG.CKT12
- net TRAC_LED: now also ABOX_HARN_2.CKT4; no longer ABOX_HARN.CKT12
- net TRA_CTL_LED: now also DSW_LG_1.CKT1; no longer DSW_LG.CKT5
- net TRA_CTL_POT: now also ABOX_HARN_2.CKT2, DSW_LG_1.CKT3; no longer ABOX_HARN.CKT10, DSW_LG.CKT7
- net TRA_CTL_SW: now also ABOX_HARN_2.CKT1; no longer ABOX_HARN.CKT9
- net TRA_CTL_SW_12: now also DSW_LG_0.CKT4; no longer DSW_LG.CKT4
- net VIN: now also DSW_LG_0.CKT1; no longer DSW_LG.CKT1
Routing:
- net VIN: track 11.2 -> 255.2 mm, vias 0 -> 4
- net A7: track 5.21 -> 140.4 mm
- net D24: track 8.55 -> 140.1 mm
- net 5V: track 243.4 -> 333.8 mm, vias 1 -> 4
- net SW1: track 0.00 -> 89.9 mm, vias 0 -> 1
- net TRA_CTL_LED: track 0.00 -> 89.4 mm
- net SHFT_D: track 0.00 -> 79.1 mm, vias 0 -> 1
- net TRAC_LED: track 0.00 -> 71.6 mm, vias 0 -> 1
- net D23: track 8.67 -> 73.3 mm, vias 0 -> 1
- net LAUNCH_LED: track 0.00 -> 62.4 mm, vias 0 -> 1
- net TRA_CTL_SW_12: track 0.00 -> 61.4 mm, vias 0 -> 1
- net D22: track 8.75 -> 67.3 mm, vias 0 -> 1
- net LAUNCHSW_LED: track 0.00 -> 57.3 mm, vias 0 -> 1
- net MODE1: track 0.00 -> 55.6 mm
- net E_DSEN_LED: track 0.00 -> 54.9 mm
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Other:
- board size 113 x 96.5 mm -> 113 x 88.9 mm
- board text added: "ABOX_HARN_0"
- board text added: "ABOX_HARN_1"
- board text added: "ABOX_HARN_2"
- board text added: "ABOX_HARN_3"
- board text added: "ABOX_PWR"
- board text added: "CD4504BE"
- board text added: "CD4504BE1"
- board text added: "DSW_LG_0"
- board text added: "DSW_LG_1"
- board text added: "DSW_LG_2"
- board text added: "JP1"
- board text added: "JP10"
- board text added: "JP11"
- board text added: "JP12"
- board text added: "JP13"
- board text added: "JP14"
- board text added: "JP15"
- board text added: "JP16"
- board text added: "JP17"
- board text added: "JP18"
- board text added: "JP2"
- board text added: "JP20"
- board text added: "JP21"
- board text added: "JP22"
- board text added: "JP23"
- board text added: "JP24"
- board text added: "JP25"
- board text added: "JP26"
- board text added: "JP27"
- board text added: "JP3"
- board text added: "JP4"
- board text added: "JP5"
- board text added: "JP6"
- board text added: "JP7"
- board text added: "JP8"
- board text added: "JP9"
- board text added: "LCD_0"
- board text added: "LCD_1"
- board text added: "LED2"
- board text added: "LED3"
- board text added: "MHybrid Dashboard Rev0.1 Brian Margosian '15"
- board text added: "Q1"
- board text added: "Q2"
- board text added: "Q4"
- board text added: "Q5"
- board text added: "R1"
- board text added: "R10"
- board text added: "R11"
- board text added: "R12"
- board text added: "R13"
- board text added: "R14"
- board text added: "R15"
- board text added: "R16"
- board text added: "R2"
- board text added: "R3"
- board text added: "R4"
- board text added: "R5"
- board text added: "R6"
- board text added: "R7"
- board text added: "R8"
- board text added: "R9"
- board text added: "S1"
