File: eagle/Control Unit/CU.brd (EAGLE design)
At the start: 116.8 x 223.5 mm, 62 parts, among them IC3 NE555, IC4 4081N

Commit message: added dash code and updated docs
Routing:
- net VBATT_FUSED: track 2019.5 -> 545.7 mm
- net GND: track 2354.7 -> 888.6 mm
- net VSENS: track 1458.4 -> 735.9 mm
- net CAN_H_L: track 556.0 -> 126.7 mm
- net E-DSNG_LED: track 804.6 -> 418.7 mm
- net GFD_RESET_SW: track 603.4 -> 220.6 mm
- net TRACTL_POT: track 682.3 -> 303.7 mm
- net LAUNCH_LED: track 686.1 -> 311.6 mm
- net TRACTL_LED: track 664.4 -> 298.2 mm
- net TRACTL_SW: track 682.9 -> 320.8 mm
- net PADDLE_DN: track 618.3 -> 260.3 mm
- net PADDLE_UP: track 618.8 -> 264.9 mm
- net N$30: track 441.5 -> 111.8 mm
- net N$31: track 437.5 -> 111.8 mm
- net N$32: track 433.6 -> 111.8 mm
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
Commit message: updated old CU and pdfs
Connections:
- removed net N$40: TS.1, TS_L.CKT1
- removed net N$44: TS.5, TS_R.CKT1
- net N$48: now also TS.1, TS_L.CKT1
- net N$49: now also TS.5, TS_R.CKT1
Routing:
- net N$49: track 9.27 -> 32.3 mm, vias 0 -> 1
- net N$44: track 23.1 -> 0.00 mm, vias 1 -> 0
- net N$48: track 8.91 -> 28.4 mm
- net N$40: track 19.5 -> 0.00 mm
Changed lines of the file:
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@@
 <wire x1="19.2786" y1="207.6958" x2="19.4056" y2="207.6958" width="0" layer="19" extent="1-1"/>
-</signal>
-<signal name="N$44">
-<contactref element="TS_R" pad="CKT1"/>
-<contactref element="TS" pad="5"/>
-<wire x1="93.98" y1="215.9" x2="93.98" y2="207.772" width="1.27" layer="16"/>
-<wire x1="99.568" y1="215.9" x2="93.98" y2="215.9" width="1.27" layer="16"/>
-<wire x1="102.616" y1="212.852" x2="99.568" y2="215.9" width="1.27" layer="16"/>
-<wire x1="102.616" y1="212.852" x2="102.9462" y2="212.6742" width="1.27" layer="16"/>
-<wire x1="91.948" y1="204.724" x2="91.44" y2="204.724" width="1.27" layer="1"/>
-<wire x1="93.98" y1="206.756" x2="91.948" y2="204.724" width="1.27" layer="1"/>
-<wire x1="93.98" y1="207.772" x2="93.98" y2="206.756" width="1.27" layer="1"/>
-<wire x1="91.44" y1="204.724" x2="91.44" y2="204.47" width="1.27" layer="1"/>
-<via x="93.98" y="207.772" extent="1-16" drill="0.508"/>
 </signal>
 <signal name="VSENS_UNFUSED">
@@
 <wire x1="37.084" y1="85.344" x2="36.83" y2="85.09" width="1.27" layer="16"/>
 <wire x1="34.544" y1="91.948" x2="34.9758" y2="92.3544" width="1.27" layer="16"/>
+<contactref element="TS" pad="1"/>
+<contactref element="TS_L" pad="CKT1"/>
+<wire x1="91.44" y1="214.63" x2="92.075" y2="214.63" width="1.27" layer="1"/>
+<wire x1="92.075" y1="214.63" x2="93.98" y2="212.725" width="1.27" layer="1"/>
+<wire x1="93.98" y1="212.725" x2="93.98" y2="212.09" width="1.27" layer="1"/>
+<wire x1="93.98" y1="212.09" x2="95.377" y2="210.5406" width="1.27" layer="1"/>
+<wire x1="95.377" y1="210.5406" x2="99.187" y2="210.5406" width="1.016" layer="1"/>
+<wire x1="99.187" y1="210.5406" x2="100.33" y2="209.55" width="1.27" layer="1"/>
+<wire x1="100.33" y1="209.55" x2="100.33" y2="205.1304" width="1.27" layer="1"/>
+<wire x1="100.33" y1="205.1304" x2="102.9462" y2="202.5142" width="1.27" layer="1"/>
+<wire x1="102.9462" y1="202.5142" x2="34.9758" y2="92.3544" width="0" layer="19" extent="1-1"/>
 </signal>
 <signal name="N$49">
@@
 <wire x1="39.116" y1="91.948" x2="39.116" y2="90.932" width="1.27" layer="1"/>
 <wire x1="39.116" y1="91.948" x2="39.1922" y2="92.3544" width="1.27" layer="1"/>
+<contactref element="TS_R" pad="CKT1"/>
+<contactref element="TS" pad="5"/>
+<wire x1="93.98" y1="215.9" x2="93.98" y2="207.772" width="1.27" layer="16"/>
+<wire x1="99.568" y1="215.9" x2="93.98" y2="215.9" width="1.27" layer="16"/>
+<wire x1="102.616" y1="212.852" x2="99.568" y2="215.9" width="1.27" layer="16"/>
+<wire x1="102.616" y1="212.852" x2="102.9462" y2="212.6742" width="1.27" layer="16"/>
+<wire x1="91.948" y1="204.724" x2="91.44" y2="204.724" width="1.27" layer="1"/>
+<wire x1="93.98" y1="206.756" x2="91.948" y2="204.724" width="1.27" layer="1"/>
+<wire x1="93.98" y1="207.772" x2="93.98" y2="206.756" width="1.27" layer="1"/>
+<wire x1="91.44" y1="204.724" x2="91.44" y2="204.47" width="1.27" layer="1"/>
+<via x="93.98" y="207.772" extent="1-16" drill="0.508"/>
+<wire x1="91.44" y1="204.47" x2="39.1922" y2="92.3544" width="0" layer="19" extent="1-1"/>
 </signal>
 <signal name="INV_ING_L">
@@
 <wire x1="19.812" y1="85.344" x2="19.4056" y2="84.9122" width="1.27" layer="16"/>
 </signal>
-<signal name="N$40">
-<contactref element="TS" pad="1"/>
-<contactref element="TS_L" pad="CKT1"/>
-<wire x1="91.44" y1="214.63" x2="92.075" y2="214.63" width="1.27" layer="1"/>
-<wire x1="92.075" y1="214.63" x2="93.98" y2="212.725" width="1.27" layer="1"/>
-<wire x1="93.98" y1="212.725" x2="93.98" y2="212.09" width="1.27" layer="1"/>
-<wire x1="93.98" y1="212.09" x2="95.377" y2="210.5406" width="1.27" layer="1"/>
-<wire x1="95.377" y1="210.5406" x2="99.187" y2="210.5406" width="1.016" layer="1"/>
-<wire x1="99.187" y1="210.5406" x2="100.33" y2="209.55" width="1.27" layer="1"/>
-<wire x1="100.33" y1="209.55" x2="100.33" y2="205.1304" width="1.27" layer="1"/>
-<wire x1="100.33" y1="205.1304" x2="102.9462" y2="202.5142" width="1.27" layer="1"/>
-</signal>
 <signal name="N$7">
