File: eagle/CAN Module/v1/CAN Module.brd (EAGLE design)
At the start: 39.4 x 33 mm, 19 parts, among them J1 AVR_SPI_PRG_6NS, Q1 16MHz, Q2 16MHz, U1 MCP2551-SN

Commit message: Rearranged files in prep for 2015
Parts:
- removed C2: 220uF, SparkFun-Capacitors:EIA3216-KIT
- removed CAN_RESISTOR: 120, SparkFun-Resistors:0805
- removed EN_CAN_RESIST: SOLDERJUMPERTRACE, SparkFun-Passives:SJ_2S-TRACE
- added C6: 100nF, SparkFun-Capacitors:0805
- added PWR, RX, TX: (no value), adafruit:CHIPLED_0805
- added R3: 4.7k, SparkFun-Resistors:0805
- added R4, R5, R6: 1k, SparkFun-Resistors:0805
- moved C5 7.12 mm to (8.13, 14.0), turned to 90 degrees
Connections:
- removed net N$4: CAN_RESISTOR.1, EN_CAN_RESIST.2
- new net N$15: R3.2, U1.8
- new net N$16: PWR.A, R4.2
- new net N$17: R5.2, TX.A
- new net N$18: R6.2, RX.A
- net 5V: now also C6.2, R4.1, R5.1, R6.1; no longer C2.A
- net CANH: no longer CAN_RESISTOR.2
- net CANL: no longer EN_CAN_RESIST.1
- net GND: now also C6.1, PWR.C, R3.1; no longer C2.C, U1.8
- net N$2: now also RX.C
- net N$3: now also TX.C
Routing:
- net N$15: track 0.00 -> 12.8 mm
- net CANL: track 13.8 -> 6.32 mm
- net RESET: track 85.5 -> 78.6 mm
- net CANH: track 10.9 -> 5.92 mm
- net N$4: track 3.31 -> 0.00 mm
- net N$17: track 0.00 -> 2.69 mm
- net N$2: track 7.54 -> 10.1 mm
- net N$16: track 0.00 -> 2.27 mm
- net GND: track 62.8 -> 61.2 mm, vias 10 -> 12
- net 5V: track 35.7 -> 37.1 mm
- net N$11: track 4.24 -> 5.17 mm
