File: eagle/CAN Module/v1/CAN Module.sch (EAGLE design)
At the start: 19 parts, among them J1 AVR_SPI_PRG_6NS, Q1 16MHz, Q2 16MHz, U1 MCP2551-SN

Commit message: Rearranged files in prep for 2015
Parts:
- removed C2: 220uF, SparkFun-Capacitors:CAP_POL1206-KIT
- removed CAN_RESISTOR: 120, SparkFun-Resistors:RESISTOR0805-RES
- removed EN_CAN_RESIST: SOLDERJUMPERNC2, SparkFun-Passives:SOLDERJUMPERNC2
- added C6: 100nF, SparkFun-Capacitors:CAP0805
- added PWR, RX, TX: (no value), adafruit:LEDCHIPLED_0805
- added R3: 4.7k, SparkFun-Resistors:RESISTOR0805-RES
- added R4, R5, R6: 1k, SparkFun-Resistors:RESISTOR0805-RES
Connections:
- removed net N$4: CAN_RESISTOR.1, EN_CAN_RESIST.2
- new net N$15: R3.2, U1.RS
- new net N$16: PWR.A, R4.2
- new net N$17: R5.2, TX.A
- new net N$18: R6.2, RX.A
- net 5V: now also C6.2, R4.1, R5.1, R6.1; no longer C2.+
- net CANH: no longer CAN_RESISTOR.2
- net CANL: no longer EN_CAN_RESIST.1
- net GND: now also C6.1, PWR.C, R3.1; no longer C2.-, U1.RS
- net N$2: now also RX.C
- net N$3: now also TX.C
